File: SignalMast-ColorLight-DualHead_array.brd (EAGLE design)
At the start: 103.5 x 104.1 mm, 97 parts

Commit message: normalized values
Parts:
- BOARD1: value BOARD100X100-NOHOLES -> BOARD
- LOWER, LOWER1, LOWER10, LOWER11, LOWER2, LOWER3, LOWER4, LOWER5, LOWER6, LOWER7, LOWER8, LOWER9, UPPER, UPPER1, UPPER10, UPPER11, UPPER2, UPPER3, UPPER4, UPPER5, UPPER6, UPPER7, UPPER8, UPPER9: value 1x4 0.100 -> 0.100
- turned LED1 to 0 degrees
- turned LED10 to 0 degrees
- turned LED11 to 0 degrees
- turned LED12 to 0 degrees
- turned LED13 to 0 degrees
- turned LED14 to 0 degrees
- turned LED15 to 0 degrees
- turned LED16 to 0 degrees
- turned LED17 to 0 degrees
- turned LED18 to 0 degrees
- turned LED19 to 0 degrees
- turned LED2 to 0 degrees
- turned LED20 to 0 degrees
- turned LED21 to 0 degrees
- turned LED22 to 0 degrees
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